File: Drive Board/Microcontroller.kicad_sch (KiCad schematic)
At the start: 0 parts

Commit message: Rev A of PCB
Parts:
- added C32, C35, C36: 1uF, Capacitor_SMD:C_0603_1608Metric_Pad1.08x0.95mm_HandSolder, symbol Device:C
- added C33, C34: 10pF, Capacitor_SMD:C_0603_1608Metric_Pad1.08x0.95mm_HandSolder, symbol Device:C
- added C37, C45: 0.1uF, Capacitor_SMD:C_0603_1608Metric_Pad1.08x0.95mm_HandSolder, symbol Device:C
- added C44, C47, C48: 100n, Capacitor_SMD:C_0603_1608Metric_Pad1.08x0.95mm_HandSolder, symbol Device:C
- added C46: 4.7uF, Capacitor_SMD:C_0603_1608Metric_Pad1.08x0.95mm_HandSolder, symbol Device:C
- added D2: LED_G, LED_SMD:LED_0805_2012Metric_Pad1.15x1.40mm_HandSolder, symbol Device:LED
- added D3: LED_O, LED_SMD:LED_0805_2012Metric_Pad1.15x1.40mm_HandSolder, symbol Device:LED
- added D4: LED, LED_SMD:LED_0805_2012Metric_Pad1.15x1.40mm_HandSolder, symbol Device:LED
- added JP1: Jumper_3_Open, Connector_PinHeader_2.54mm:PinHeader_1x03_P2.54mm_Vertical, symbol Jumper:Jumper_3_Open
- added JP2: Jumper_2_Open, Connector_PinHeader_2.54mm:PinHeader_1x02_P2.54mm_Vertical, symbol Jumper:Jumper_2_Open
- added R27: 10K, Resistor_SMD:R_0603_1608Metric_Pad0.98x0.95mm_HandSolder, symbol Device:R
- added R28, R29, R30: 1k, Resistor_SMD:R_0603_1608Metric_Pad0.98x0.95mm_HandSolder, symbol Device:R
- added R31: 120, Resistor_SMD:R_0603_1608Metric_Pad0.98x0.95mm_HandSolder, symbol Device:R
- added R32, R39, R42: 10k, Resistor_SMD:R_0603_1608Metric_Pad0.98x0.95mm_HandSolder, symbol Device:R
- added SW1, SW2: SW_Push, Footprints:SKRPADE010_AAL, symbol Switch:SW_Push
- added SW4: SW_DIP_x05, Footprints:SW5_219SMT, symbol Switch:SW_DIP_x05
- added U4: TLV75533PDBVR, Package_TO_SOT_SMD:SOT-23-5, symbol Regulator_Linear:TLV75533PDBV
- added U5: MCP2562-E-SN, Package_SO:SOIC-8_3.9x4.9mm_P1.27mm, symbol Interface_CAN_LIN:MCP2562-E-SN
- added U6: ~, Package_QFP:LQFP-48_7x7mm_P0.5mm, symbol UGRT_ST_STM32G0:STM32G0B1CETx_Annotated
- added Y2: 8MHz, Footprints:XTAL_ECS-80-8-30Q-VS-TR, symbol Device:Crystal
Connections:
- new net: C34.1, U6.9 (PF1-OSC_OUT), Y2.1
- new net: C33.2, U6.8 (PF0-OSC_IN), Y2.2
- new net: JP2.2 (B), R31.1
- new net: D4.2 (A), R30.1
- new net: D2.2 (A), R28.2
- new net: JP1.2 (C), U6.36 (PA14)
- new net: SW4.5, U6.42 (PB3)
- new net: SW4.4, U6.43 (PB4)
- new net: SW4.3, U6.44 (PB5)
- new net: SW4.2, U6.45 (PB6)
- new net: SW4.1, U6.46 (PB7)
- new net: JP1.3 (B), R27.1, SW1.1
- new net: D3.2 (A), R29.2
- new net +3V3: C32.1, C36.1, C44.1, C46.1, C47.1, C48.1, R28.1, R29.1, R30.2, R32.2, R39.2, R42.2, SW1.2, SW4.10, SW4.6, SW4.7, SW4.8, SW4.9, U4.5 (OUT), U5.5 (Vio), U6.4 (VBAT), U6.5 (VREF+), U6.6 (VDD/VDDA)
- new net +5V: C35.1, C37.1, U4.1 (IN), U4.3 (EN), U5.3 (VDD)
- new net BLDC EN_GATE: U6.37 (PA15)
- new net BLDC INH_A: U6.28 (PA8)
- new net BLDC INH_B: U6.33 (PA9/PA11)
- new net BLDC INH_C: U6.34 (PA10/PA12)
- new net BLDC INL_A: U6.25 (PB13)
- new net BLDC INL_B: U6.26 (PB14)
- new net BLDC INL_C: U6.27 (PB15)
- new net BLDC NFault: R32.1, U6.40 (PD2)
- new net BLDC OCTW: R39.1, U6.41 (PD3)
- new net BLDC SO1: U6.19 (PB0)
- new net BLDC SO2: U6.20 (PB1)
- new net BOOT: C45.1, SW2.2, U6.10 (PF2-NRST)
- new net Brake_IN1: U6.11 (PA0)
- new net Brake_IN2: U6.12 (PA1)
- new net CANH: JP2.1 (A), U5.7 (CANH)
- new net CANL: R31.2, U5.6 (CANL)
- new net DC_CAL: U6.48 (PB9)
- new net EncoderA_DO: U6.16 (PA5)
- new net EncoderA_PROG: U6.17 (PA6)
- new net EncoderB_DO: U6.14 (PA3)
- new net EncoderB_PROG: U6.13 (PA2)
- new net Encoder_CLK: U6.15 (PA4)
- new net FDCAN1_RX: D2.1 (K), U5.4 (RXD), U6.38 (PD0)
- new net FDCAN1_TX: D3.1 (K), U5.1 (TXD), U6.39 (PD1)
- new net GND: C32.2, C33.1, C34.2, C35.2, C36.2, C37.2, C44.2, C45.2, C46.2, C47.2, C48.2, D4.1 (K), R27.2, SW2.1, U4.2 (GND), U5.2 (VSS), U5.8 (STBY), U6.7 (VSS/VSSA)
- new net MUXA: U6.1 (PC13)
- new net MUXB: U6.2 (PC14-OSC32_IN)
- new net MUXC: U6.3 (PC15-OSC32_OUT)
- new net PWRGD: R42.1, U6.47 (PB8)
- new net SWCLK: JP1.1 (A)
- new net SWDIO: U6.35 (PA13)
- new net Steer_IN1: U6.30 (PC6)
- new net Steer_IN2: U6.31 (PC7)
- new net Temp Output: U6.22 (PB10)
- no-connect marks 0 -> 6
Other:
- note added: "CANFD Transceiver"
- note added: "HSE"
- note added: "LDO (5V -> 3V3)"
- note added: "LSE"
- note added: "STM32G0B1CET6 General"
- note added: "Software-Compatible Pull-Down/Up Network"
