File: Drive Board/Steer Angle Brake Motor.kicad_sch (KiCad schematic)
At the start: 0 parts

Commit message: Rev A of PCB
Parts:
- added R43: 64000, Resistor_SMD:R_0603_1608Metric_Pad0.98x0.95mm_HandSolder, symbol Device:R
- added U7: DRV8231DDAR, Package_SO:Texas_HTSOP-8-1EP_3.9x4.9mm_P1.27mm_EP2.95x4.9mm_Mask2.4x3.1mm_ThermalVias, symbol Robotics_club:DRV8871DDA_1
Connections:
- new net: R43.1, U7.4 (ILIM)
- new net +12V: U7.5 (VM)
- new net Brake_IN1: U7.3 (IN1)
- new net Brake_IN2: U7.2 (IN2)
- new net Brake_OUT1: U7.8 (OUT2)
- new net Brake_OUT2: U7.6 (OUT1)
- new net GND: R43.2, U7.1 (GND), U7.7 (PGND)
