File: Drive Board/Steer Angle Motor.kicad_sch (KiCad schematic)
At the start: 0 parts

Commit message: Rev A of PCB
Parts:
- added R44: 64000, Resistor_SMD:R_0603_1608Metric_Pad0.98x0.95mm_HandSolder, symbol Device:R
- added U8: DRV8231DDAR, Package_SO:Texas_HTSOP-8-1EP_3.9x4.9mm_P1.27mm_EP2.95x4.9mm_Mask2.4x3.1mm_ThermalVias, symbol Robotics_club:DRV8871DDA_1
Connections:
- new net: R44.1, U8.4 (ILIM)
- new net +12V: U8.5 (VM)
- new net GND: R44.2, U8.1 (GND), U8.7 (PGND)
- new net Steer_IN1: U8.3 (IN1)
- new net Steer_IN2: U8.2 (IN2)
- new net Steer_OUT1: U8.8 (OUT2)
- new net Steer_OUT2: U8.6 (OUT1)
