File: Drive Board/Voltage Rails.kicad_sch (KiCad schematic)
At the start: 0 parts

Commit message: Rev A of PCB
Other:
- note added: "Protections circuitry??"
Changed lines of the file:
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@@
 	(generator_version "9.0")
 	(paper "A4")
+	(text "Protections circuitry??"
+		(exclude_from_sim no)
+		(at 175.768 99.568 0)
+		(effects
+			(font
+				(size 1.27 1.27)
+			)
+		)
+	)
 )
