File: Drive Board/Drive Board.kicad_pcb (KiCad board)
At the start: 2 copper layers, 70 x 63 mm, 136 parts, among them J1 1984620, J10 B5B-XH-A, J11 Conn_01x04, J2 1984617, J3 1984617, J4 1984617, J5 B2B-XH-A, J6 B3B-XH-A, J7 B2B-XH-A, J8 B2B-XH-A, J9 B5B-XH-A, Q10 SQD70140EL_GE3, Q11 SQD70140EL_GE3, Q6 SQD70140EL_GE3, Q7 SQD70140EL_GE3, Q8 SQD70140EL_GE3, Q9 SQD70140EL_GE3, SW1 SW_Push, SW2 SW_Push, SW4 SW_DIP_x05, U1 DRV8302DCAR, U2 CD4051B, U3 LM2678SX-12_NOPB, U4 TLV75533PDBVR, U5 MCP2562-E-SN, U7 DRV8231DDAR, U8 DRV8231DDAR, Y2 8MHz

Commit message: finished RV1 of board
Parts:
- added G***: LOGO, Footprints:UGRT_Logo, F.Cu at (84.3, 91.9)
- moved C14 157.8 mm to (165.6, 151.1), turned to -90 degrees
- moved C20 157.7 mm to (165.6, 146.8), turned to -90 degrees
- moved C22 153.4 mm to (163.4, 146.8), turned to 90 degrees
- moved C21 150.6 mm to (164.4, 135.8), turned to 90 degrees
- moved J4 149.0 mm to (161.8, 68.8), turned to 180 degrees
- moved R10 144.0 mm to (154.4, 151.1), turned to -90 degrees
- moved R38 141.7 mm to (163.4, 151.2), turned to 90 degrees
- moved C26 140.6 mm to (162.0, 127.2), turned to 90 degrees
- moved R36 140.5 mm to (158.9, 151.2), turned to 90 degrees
- moved C18 140.2 mm to (149.7, 151.1), turned to -90 degrees
- moved R19 139.7 mm to (152.0, 151.1), turned to 90 degrees
- moved C17 139.5 mm to (149.7, 146.9), turned to 90 degrees
- moved R40 138.5 mm to (161.2, 151.2), turned to 90 degrees
- moved R35 137.5 mm to (156.6, 146.8), turned to -90 degrees
- moved R34 137.1 mm to (154.4, 146.9), turned to -90 degrees
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Connections:
- C8 pad 1: +3.3V -> +3V3
- J11 pad 1: +3.3V -> +3V3
- J6 pad 1: BOOT -> CANL
- J6 pad 3: CANL -> BOOT
- R1 pad 1: +3.3V -> +3V3
- R2 pad 1: +3.3V -> +3V3
- R3 pad 1: +3.3V -> +3V3
- R4 pad 1: +3.3V -> +3V3
- R5 pad 1: +3.3V -> +3V3
- R6 pad 1: +3.3V -> +3V3
- R7 pad 1: +3.3V -> +3V3
- U1 pad 24: +3.3V -> +3V3
- U2 pad 16: +3.3V -> +3V3
Routing:
- net GND: track 0.00 -> 137.2 mm, vias 0 -> 143
- net BLDC A: track 0.00 -> 88.7 mm, vias 0 -> 2
- net +3V3: track 0.00 -> 87.6 mm, vias 0 -> 25
- net /BLDC Control/SN2: track 0.00 -> 85.5 mm, vias 0 -> 2
- net /Temperature Measurement/Temp Motor Driver BLDC: track 0.00 -> 85.5 mm, vias 0 -> 2
- net BOOT: track 0.00 -> 79.5 mm, vias 0 -> 1
- net /BLDC Control/SN1: track 0.00 -> 72.3 mm, vias 0 -> 2
- net Net-(U1-BST_A): track 0.00 -> 69.0 mm, vias 0 -> 2
- net /Temperature Measurement/Temp Motor Driver Steering: track 0.00 -> 66.3 mm, vias 0 -> 2
- net Brake_IN1: track 0.00 -> 65.1 mm, vias 0 -> 2
- net Brake_IN2: track 0.00 -> 64.0 mm, vias 0 -> 2
- net Net-(U1-GH_A): track 0.00 -> 61.2 mm, vias 0 -> 2
- net Net-(U1-GL_A): track 0.00 -> 60.7 mm, vias 0 -> 2
- net /Temperature Measurement/Temp Motor Driver Brake: track 0.00 -> 58.8 mm, vias 0 -> 2
- net Temp Output: track 0.00 -> 58.5 mm, vias 0 -> 2
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- added copper zone on F.Cu, net +12V
- added copper zone on In2.Cu, net +12V
- added copper zone on F.Cu, net +24V
- added copper zone on In2.Cu, net +24V
- added copper zone on F.Cu, net +3V3
- added copper zone on In2.Cu, net +3V3
- added copper zone on F.Cu, net +5V
- added copper zone on In2.Cu, net +5V
- added copper zone on F.Cu, net /BLDC Control/SN1
- added copper zone on F.Cu, net /BLDC Control/SN2
- added copper zone on F.Cu, net /BLDC Control/SW Node
- added copper zone on F.Cu, net BLDC A
- added copper zone on F.Cu, net BLDC B
- added copper zone on F.Cu, net BLDC C
- added copper zone on F.Cu, net Brake_OUT1
- added copper zone on F.Cu, net Brake_OUT2
- added copper zone on F.Cu, net GND
- added copper zone on In1.Cu, net GND
- added copper zone on F.Cu, net Net-(D5-K)
- added copper zone on F.Cu, net Steer_OUT1
- added copper zone on F.Cu, net Steer_OUT2
Other:
- board size 70 x 63 mm -> 93.5 x 89.3 mm
- copper layers 2 -> 4
- board text added: "24V"
- board text added: "3v3"
- board text added: "A"
- board text added: "B"
- board text added: "BLDC"
- board text added: "BLDC_T"
- board text added: "BM_T"
- board text added: "BOOT"
- board text added: "BrakeMotor"
- board text added: "C"
- board text added: "CAN"
- board text added: "CLK"
- board text added: "DIO"
- board text added: "Drive Board RV1"
- board text added: "GND"
- board text added: "H"
- board text added: "Kavin Chris Daniel"
- board text added: "L"
- board text added: "RESET"
- board text added: "SteerMotor"
- board text added: "Steer_T"
