File: Drive Board/Drive Board.kicad_sch (KiCad schematic)
At the start: 0 parts

Commit message: Rev A of PCB
Other:
- removed sheet Voltage Rails
- added sheet Secondary Power Rail (Secondary Power Rail.kicad_sch)
