File: Power Board Revisions/PDB_V3/PDB_V3.kicad_sch (KiCad schematic)
At the start: 5 parts, among them J2 Conn_01x02

Commit message: Finalized PDB V3 for first design review
Other:
- note added: "12V Channel"
- note added: "24V Channel"
- note added: "5V Channel"
- note added: "Main Connectors"
- note added: "Mounting"
- company: (none) -> University of Guelph Robotics Team
- title: (none) -> Power Distribution Board V3
- moved on the sheet: H1, H2, H3, H4, J2
