File: Power Board Revisions/PDB_V3/PDB_V3.kicad_pcb (KiCad board)
At the start: 2 copper layers, 199 x 114.5 mm, 212 parts, among them J1 1017507, J2 Conn_01x02, J3 1017507, J4 1017507, J5 1017507, Q1_1 NMOS, Q1_2 NMOS, Q1_2_1 NMOS, Q1_2_2 NMOS, Q1_2_3 NMOS, Q1_3 NMOS, Q1_4 NMOS, Q2_1 NMOS, Q2_2 NMOS, Q2_3 NMOS, Q2_4 NMOS, Q3_1 NMOS, Q3_2 NMOS, Q3_2_1 NMOS, Q3_2_2 NMOS, Q3_2_3 NMOS, Q3_2_4 NMOS, Q3_3 NMOS, Q3_4 NMOS, Q4_1 NMOS, Q4_2 NMOS, Q4_3 NMOS, Q4_4 NMOS, SW1 SW_SPST, SW10 SW_SPST, SW11 SW_SPST, SW12 SW_SPST, SW13 SW_SPST, SW14 SW_SPST, SW15 SW_SPST, SW16 SW_SPST, SW17 SW_SPST, SW18 SW_SPST, SW19 SW_SPST, SW2 SW_SPST, SW20 SW_SPST, SW21 SW_SPST, SW22 SW_SPST, SW23 SW_SPST, SW24 SW_SPST, SW3 SW_SPST, SW4 SW_SPST, SW5 SW_SPST, SW6 SW_SPST, SW7 SW_SPST, SW8 SW_SPST, SW9 SW_SPST, U1 LM5176QPWPRQ1, U2 LM5176QPWPRQ1, U3 LM5176QPWPRQ1, U4 LM5176QPWPRQ1

Commit message: Updated PDB V3
Parts:
- moved J2 33.1 mm to (102.5, 70.2)
- moved Cbulk1 24.9 mm to (200.7, 36.9)
- moved Cin1 24.9 mm to (186.9, 36.9)
- moved Q3_2_1 24.9 mm to (191.8, 57.3)
- moved Ruvb1 24.9 mm to (164.9, 38.5)
- moved Ruvt1 24.9 mm to (164.9, 36.0)
- moved U1 24.9 mm to (176.4, 54.5)
- moved Cbias1 24.9 mm to (170.1, 69.0)
- moved Cboot1_1 24.9 mm to (178.9, 46.5)
- moved Cboot2_1 24.9 mm to (181.6, 46.5)
- moved Ccomp1_1 24.9 mm to (164.9, 63.5)
- moved Ccomp2_1 24.9 mm to (164.9, 61.0)
- moved Ccs1 24.9 mm to (174.1, 62.8)
- moved Cdith1 24.9 mm to (164.9, 51.0)
- moved Cf1 24.9 mm to (164.9, 41.0)
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Routing:
- net /lm5176 12v Channel 1/SW2_1: track 75.7 -> 72.0 mm
Other:
- board size 199 x 114.5 mm -> 199 x 146.3 mm

Commit message: Updated PDB V3
I dislike KiCad on windows
Parts:
- added F25: Fuse, Footprints:FUSE_3557-2, F.Cu at (207.8, 90.5)
- added F26: Fuse, Footprints:FUSE_3557-2, F.Cu at (207.8, 98.0)
- added F27: Fuse, Footprints:FUSE_3557-2, F.Cu at (207.5, 151.5)
- added F28: Fuse, Footprints:FUSE_3557-2, F.Cu at (207.5, 159.0)
- added F29: Fuse, Footprints:FUSE_3557-2, F.Cu at (-78.3, 201.3)
- added F30: Fuse, Footprints:FUSE_3557-2, F.Cu at (-85.8, 201.3)
- added F31: Fuse, Footprints:FUSE_3557-2, F.Cu at (-182.3, -34.8)
- added F32: Fuse, Footprints:FUSE_3557-2, F.Cu at (-189.8, -34.8)
- added SW25: SW_SPST, Footprints:ESwitch 1101A4CQEA, F.Cu at (225.3, 90.5)
- added SW26: SW_SPST, Footprints:ESwitch 1101A4CQEA, F.Cu at (225.3, 98.0)
- added SW27: SW_SPST, Footprints:ESwitch 1101A4CQEA, F.Cu at (225.0, 151.5)
- added SW28: SW_SPST, Footprints:ESwitch 1101A4CQEA, F.Cu at (225.0, 159.0)
- added SW29: SW_SPST, Footprints:ESwitch 1101A4CQEA, F.Cu at (-78.3, 218.8)
- added SW30: SW_SPST, Footprints:ESwitch 1101A4CQEA, F.Cu at (-85.8, 218.8)
- added SW31: SW_SPST, Footprints:ESwitch 1101A4CQEA, F.Cu at (-182.3, -17.3)
- added SW32: SW_SPST, Footprints:ESwitch 1101A4CQEA, F.Cu at (-189.8, -17.3)
- J1, J3, J4, J5: value 1017507 -> 1862262; footprint Footprints:Phoenix 1017507 -> Footprints:PHOENIX 1862262
- moved F4 227.9 mm to (-137.3, -34.8), turned to 90 degrees
- moved F8 227.5 mm to (-144.7, -34.8), turned to 90 degrees
- moved F12 227.1 mm to (-152.2, -34.8), turned to 90 degrees
- moved F16 226.7 mm to (-159.7, -34.8), turned to 90 degrees
- moved F20 226.3 mm to (-167.2, -34.8), turned to 90 degrees
- moved F24 226.0 mm to (-174.7, -34.8), turned to 90 degrees
- moved SW4 196.4 mm to (-137.3, -17.1), turned to 90 degrees
- moved SW8 196.0 mm to (-144.8, -17.0), turned to 90 degrees
- moved SW12 195.7 mm to (-152.3, -17.1), turned to 90 degrees
- moved SW16 195.4 mm to (-159.8, -17.1), turned to 90 degrees
- moved SW20 195.0 mm to (-167.3, -17.1), turned to 90 degrees
- moved SW24 194.8 mm to (-174.8, -17.3), turned to 90 degrees
- moved J5 187.0 mm to (-192.3, 1.74)
- moved J4 172.7 mm to (-88.3, 237.8)
- moved SW7 144.6 mm to (-40.8, 219.0), turned to 90 degrees
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Connections:
- J1 pad 1_2: Net-(SW21-A) -> GND
- J1 pad 2_1: GND -> Net-(SW26-A)
- J1 pad 2_2: Net-(SW17-A) -> Net-(SW26-A)
- J1 pad 3_2: Net-(SW13-A) -> GND
- J1 pad 4_1: GND -> Net-(SW25-A)
- J1 pad 4_2: Net-(SW9-A) -> Net-(SW25-A)
- J1 pad 5_2: Net-(SW5-A) -> GND
- J1 pad 6_1: GND -> Net-(SW21-A)
- J1 pad 6_2: Net-(SW1-A) -> Net-(SW21-A)
- J3 pad 1_2: Net-(SW22-A) -> GND
- J3 pad 2_1: GND -> Net-(SW28-A)
- J3 pad 2_2: Net-(SW18-A) -> Net-(SW28-A)
- J3 pad 3_2: Net-(SW14-A) -> GND
- J3 pad 4_1: GND -> Net-(SW27-A)
- J3 pad 4_2: Net-(SW10-A) -> Net-(SW27-A)
- J3 pad 5_2: Net-(SW6-A) -> GND
- J3 pad 6_1: GND -> Net-(SW22-A)
- J3 pad 6_2: Net-(SW2-A) -> Net-(SW22-A)
- J4 pad 1_2: Net-(SW23-A) -> GND
- J4 pad 2_1: GND -> Net-(SW30-A)
- J4 pad 2_2: Net-(SW19-A) -> Net-(SW30-A)
- J4 pad 3_2: Net-(SW15-A) -> GND
- J4 pad 4_1: GND -> Net-(SW29-A)
- J4 pad 4_2: Net-(SW11-A) -> Net-(SW29-A)
- J4 pad 5_2: Net-(SW7-A) -> GND
- J4 pad 6_1: GND -> Net-(SW23-A)
- J4 pad 6_2: Net-(SW3-A) -> Net-(SW23-A)
- J5 pad 1_2: Net-(SW24-A) -> GND
- J5 pad 2_1: GND -> Net-(SW32-A)
- J5 pad 2_2: Net-(SW20-A) -> Net-(SW32-A)
- J5 pad 3_2: Net-(SW16-A) -> GND
- J5 pad 4_1: GND -> Net-(SW31-A)
- J5 pad 4_2: Net-(SW12-A) -> Net-(SW31-A)
- J5 pad 5_2: Net-(SW8-A) -> GND
- J5 pad 6_1: GND -> Net-(SW24-A)
- J5 pad 6_2: Net-(SW4-A) -> Net-(SW24-A)
Routing:
- net /lm5176 12v Channel 2/SW1_1: track 53.8 -> 70.8 mm
- net Net-(SW32-B): track 0.00 -> 15.9 mm
- net Net-(SW31-B): track 0.00 -> 15.9 mm
- net Net-(SW26-B): track 0.00 -> 15.9 mm
- net Net-(SW25-B): track 0.00 -> 15.9 mm
- net Net-(SW30-B): track 0.00 -> 15.9 mm
- net Net-(SW29-B): track 0.00 -> 15.9 mm
- net Net-(SW28-B): track 0.00 -> 15.9 mm
- net Net-(SW27-B): track 0.00 -> 15.9 mm
- net Net-(SW28-A): track 0.00 -> 12.7 mm
- net Net-(SW32-A): track 0.00 -> 12.7 mm
- net Net-(SW30-A): track 0.00 -> 12.7 mm
- net Net-(SW26-A): track 0.00 -> 12.7 mm
- net Net-(SW3-B): track 16.0 -> 3.40 mm
- net Net-(SW4-B): track 16.0 -> 3.40 mm
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- added copper zone on F.Cu, net /lm5176 12v Channel 1/BIAS_1
Other:
- board size 199 x 146.3 mm -> 193.8 x 137 mm
- board text added: "// ETHAN HUBER"
- board text added: "let pcb = 'Power Distro Board V3'"

Commit message: Finalized PDB V3 for first design review
Parts:
- added G***: LOGO, Dependencies:ugrt_logo, F.Cu at (145.8, 99.5)
- added G***: LOGO, LOGO, F.Cu at (146.8, 85.8)
- L1, L2, L3, L4: footprint Footprints:XAL1580 -> Footprints:WE-HCM_1411
- moved F32 279.3 mm to (82.0, 29.7), turned to 0 degrees
- moved F31 273.9 mm to (82.0, 37.2), turned to 0 degrees
- moved F24 268.8 mm to (82.0, 44.8), turned to 0 degrees
- moved F20 264.0 mm to (82.0, 52.3), turned to 0 degrees
- moved F16 259.6 mm to (82.0, 59.8), turned to 0 degrees
- moved SW32 258.6 mm to (64.5, 29.7), turned to 0 degrees
- moved F12 255.5 mm to (82.0, 67.3), turned to 0 degrees
- moved SW31 252.7 mm to (64.5, 37.2), turned to 0 degrees
- moved F8 251.8 mm to (82.0, 74.8), turned to 0 degrees
- moved F4 248.5 mm to (82.0, 82.2), turned to 0 degrees
- moved SW24 247.2 mm to (64.5, 44.7), turned to 0 degrees
- moved SW20 241.7 mm to (64.3, 52.2), turned to 0 degrees
- moved J5 239.2 mm to (45.5, 27.2), turned to -90 degrees
- moved SW16 236.9 mm to (64.3, 59.7), turned to 0 degrees
- moved SW12 232.4 mm to (64.3, 67.2), turned to 0 degrees
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Routing:
- net SW2_3: track 0.00 -> 82.6 mm, vias 0 -> 4
- net SW1_3: track 0.00 -> 63.6 mm, vias 0 -> 2
- net VOSNS_3: track 0.00 -> 59.0 mm, vias 0 -> 2
- net Net-(U3-BIAS): track 0.00 -> 40.0 mm, vias 0 -> 4
- net VCC: track 83.1 -> 119.9 mm
- net RCS_3: track 0.00 -> 29.5 mm, vias 0 -> 2
- net LDRV2_3: track 0.00 -> 25.4 mm, vias 0 -> 2
- net LDRV1_3: track 0.00 -> 24.5 mm, vias 0 -> 2
- net HDRV1_3: track 0.00 -> 24.4 mm, vias 0 -> 3
- net Net-(Dboot1_3-A): track 0.00 -> 23.2 mm, vias 0 -> 2
- net HDRV2_3: track 0.00 -> 18.8 mm, vias 0 -> 3
- net FB_3: track 0.00 -> 17.8 mm
- net Net-(U3-EN): track 0.00 -> 17.8 mm
- net Net-(U3-CSG): track 0.00 -> 16.1 mm
- net Net-(Dboot2_3-K): track 0.00 -> 15.8 mm, vias 0 -> 2
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- added copper zone on F.Cu, net VOSNS_3
Other:
- board size 193.8 x 137 mm -> 207.5 x 137 mm
- board text added: "+"
- board text added: "-"
- board text added: "12V"
- board text added: "24V"
- board text added: "5V"
- board text added: "JULY 15 2026"
- board text added: "Power Distro Board V3"
- board text removed: "let pcb = 'Power Distro Board V3'"

Commit message: Edited PDBV3: Moved capacitors to reduce hot loop size
Parts:
- moved Cin2 14.8 mm to (98.0, 135.4)
- moved Cin4 14.6 mm to (196.2, 100.8)
- moved Cin3 14.6 mm to (98.0, 72.2)
- moved Cin1 14.6 mm to (196.2, 39.1)
- moved Cf1 11.2 mm to (176.5, 48.2), turned to 180 degrees
- moved Cf4 11.1 mm to (176.2, 110.2), turned to 180 degrees
- moved Cf3 11.0 mm to (119.2, 62.5), turned to 0 degrees
- moved Cf2 10.8 mm to (119.5, 125.5), turned to 0 degrees
- moved Cbulk1 9.84 mm to (186.0, 35.9)
- moved Cbulk4 9.73 mm to (186.0, 97.5)
- moved Cbulk2 8.73 mm to (108.2, 138.5)
- moved Cbulk3 8.73 mm to (108.2, 75.2)
- moved Ruvb3 2.70 mm to (127.5, 69.5)
- moved Ruvt3 2.70 mm to (127.5, 72.0)
- moved Ruvb1 2.50 mm to (167.8, 41.2)
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Routing:
- net GND: track 58.5 -> 90.5 mm, vias 376 -> 362
- net VCC: track 119.9 -> 106.0 mm
- net Net-(U1-EN): track 18.7 -> 15.1 mm
- net Net-(U4-EN): track 18.7 -> 15.2 mm
- net Net-(U3-EN): track 17.8 -> 15.0 mm
- net Net-(U4-VIN): track 16.3 -> 14.1 mm
- net Net-(U1-VIN): track 16.3 -> 14.5 mm
- net Net-(U2-EN): track 17.8 -> 16.2 mm
- net Net-(U3-VIN): track 13.5 -> 12.6 mm
- net Net-(U2-VIN): track 13.5 -> 12.8 mm

Commit message: Updated PDB V3
Parts:
- Q3_1, Q3_2, Q3_2_1, Q3_2_2, Q3_2_3, Q3_2_4, Q3_3, Q3_4, Q4_1, Q4_2, Q4_3, Q4_4: footprint Footprints:CSD17575Q3 -> Footprints:IAUCN04S7L019
- moved Q3_2_1 5.97 mm to (199.0, 61.6)
- moved Q3_2_4 5.41 mm to (198.7, 122.9)
- moved Q3_1 4.84 mm to (199.0, 56.1)
- moved Q3_4 4.46 mm to (198.7, 117.4)
- moved Q3_2 3.74 mm to (96.0, 119.6)
- moved Q4_1 3.63 mm to (195.6, 74.5), turned to 180 degrees
- moved Q4_4 3.60 mm to (195.4, 136.5), turned to 180 degrees
- moved Q1_1 2.02 mm to (199.0, 50.6)
- moved Q1_2_1 1.90 mm to (199.0, 45.1)
- moved Q2_4 1.80 mm to (198.7, 128.4)
- moved Q2_1 1.65 mm to (199.0, 67.1)
- moved Q1_4 1.65 mm to (198.7, 111.9)
- moved Q1_2_2 1.63 mm to (198.8, 106.4)
- moved Cin1 1.27 mm to (197.5, 39.4)
- moved Cbulk1 1.26 mm to (187.2, 36.0)
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Routing:
- net VCC: track 106.0 -> 71.8 mm
- net /lm5176 12v Channel 1/HDRV2_1: track 17.5 -> 23.5 mm
- net VOSNS_3: track 59.0 -> 53.4 mm
- net VOSNS_2: track 58.8 -> 53.2 mm
- net /lm5176 12v Channel 2/SW1_1: track 63.4 -> 68.7 mm
- net /lm5176 12v Channel 1/SW2_1: track 83.0 -> 77.8 mm, vias 4 -> 5
- net /lm5176 12v Channel 2/HDRV2_1: track 17.5 -> 22.7 mm
- net /lm5176 12v Channel 1/SW1_1: track 63.4 -> 68.4 mm
- net /lm5176 12v Channel 1/HDRV1_1: track 21.9 -> 25.3 mm
- net /lm5176 12v Channel 2/HDRV1_1: track 21.9 -> 25.0 mm
- net /lm5176 12v Channel 2/LDRV2_1: track 25.5 -> 27.6 mm
- net /lm5176 12v Channel 1/LDRV2_1: track 25.5 -> 27.6 mm
- net SW1_2: track 55.7 -> 54.1 mm
- net /lm5176 12v Channel 1/LDRV1_1: track 23.7 -> 25.3 mm
- net /lm5176 12v Channel 2/SW2_1: track 82.6 -> 84.2 mm, vias 4 -> 3
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- removed copper zone on F.Cu, net VOSNS_2
