File: Power Board Revisions/PDB_V3/PDB_V3.kicad_pcb (KiCad board)
At the start: 2 copper layers, 207.5 x 137 mm, 230 parts, among them J1 1862262, J2 Conn_01x02, J3 1862262, J4 1862262, J5 1862262, Q1_1 NMOS, Q1_2 NMOS, Q1_2_1 NMOS, Q1_2_2 NMOS, Q1_2_3 NMOS, Q1_3 NMOS, Q1_4 NMOS, Q2_1 NMOS, Q2_2 NMOS, Q2_3 NMOS, Q2_4 NMOS, Q3_1 NMOS, Q3_2 NMOS, Q3_2_1 NMOS, Q3_2_2 NMOS, Q3_2_3 NMOS, Q3_2_4 NMOS, Q3_3 NMOS, Q3_4 NMOS, Q4_1 NMOS, Q4_2 NMOS, Q4_3 NMOS, Q4_4 NMOS, SW1 SW_SPST, SW10 SW_SPST, SW11 SW_SPST, SW12 SW_SPST, SW13 SW_SPST, SW14 SW_SPST, SW15 SW_SPST, SW16 SW_SPST, SW17 SW_SPST, SW18 SW_SPST, SW19 SW_SPST, SW2 SW_SPST, SW20 SW_SPST, SW21 SW_SPST, SW22 SW_SPST, SW23 SW_SPST, SW24 SW_SPST, SW25 SW_SPST, SW26 SW_SPST, SW27 SW_SPST, SW28 SW_SPST, SW29 SW_SPST, SW3 SW_SPST, SW30 SW_SPST, SW31 SW_SPST, SW32 SW_SPST, SW4 SW_SPST, SW5 SW_SPST, SW6 SW_SPST, SW7 SW_SPST, SW8 SW_SPST, SW9 SW_SPST, U1 LM5176QPWPRQ1, U2 LM5176QPWPRQ1, U3 LM5176QPWPRQ1, U4 LM5176QPWPRQ1

Commit message: Finalized PDB V3 Rev 1
Parts:
- removed Coutx1, Coutx3, Coutx4: 70uF, Capacitor_SMD:C_1206_3216Metric_Pad1.33x1.80mm_HandSolder
- removed Coutx2: 66uF, Capacitor_SMD:C_1206_3216Metric_Pad1.33x1.80mm_HandSolder
- removed the G*** at (145.8, 99.5)
- added Coutx1_1: 22uF, Capacitor_SMD:C_1206_3216Metric_Pad1.33x1.80mm_HandSolder, F.Cu at (170.0, 76.8)
- added Coutx1_2: 22uF, Capacitor_SMD:C_1206_3216Metric_Pad1.33x1.80mm_HandSolder, F.Cu at (170.0, 74.2)
- added Coutx1_3: 22uF, Capacitor_SMD:C_1206_3216Metric_Pad1.33x1.80mm_HandSolder, F.Cu at (170.0, 71.7)
- added Coutx1_4: 22uF, Capacitor_SMD:C_1206_3216Metric_Pad1.33x1.80mm_HandSolder, F.Cu at (170.0, 69.2)
- added Coutx2_1: 22uF, Capacitor_SMD:C_1206_3216Metric_Pad1.33x1.80mm_HandSolder, F.Cu at (126.3, 97.8)
- added Coutx2_2: 22uF, Capacitor_SMD:C_1206_3216Metric_Pad1.33x1.80mm_HandSolder, F.Cu at (126.3, 100.2)
- added Coutx2_3: 22uF, Capacitor_SMD:C_1206_3216Metric_Pad1.33x1.80mm_HandSolder, F.Cu at (126.3, 102.8)
- added Coutx2_4: 22uF, Capacitor_SMD:C_1206_3216Metric_Pad1.33x1.80mm_HandSolder, F.Cu at (126.3, 105.2)
- added Coutx3_1: 22uF, Capacitor_SMD:C_1206_3216Metric_Pad1.33x1.80mm_HandSolder, F.Cu at (126.5, 35.8)
- added Coutx3_2: 22uF, Capacitor_SMD:C_1206_3216Metric_Pad1.33x1.80mm_HandSolder, F.Cu at (126.5, 38.3)
- added Coutx3_3: 22uF, Capacitor_SMD:C_1206_3216Metric_Pad1.33x1.80mm_HandSolder, F.Cu at (126.5, 40.8)
- added Coutx3_4: 22uF, Capacitor_SMD:C_1206_3216Metric_Pad1.33x1.80mm_HandSolder, F.Cu at (126.5, 43.2)
- added Coutx4_1: 22uF, Capacitor_SMD:C_1206_3216Metric_Pad1.33x1.80mm_HandSolder, F.Cu at (169.0, 138.7)
- added Coutx4_2: 22uF, Capacitor_SMD:C_1206_3216Metric_Pad1.33x1.80mm_HandSolder, F.Cu at (169.0, 136.2)
- added Coutx4_3: 22uF, Capacitor_SMD:C_1206_3216Metric_Pad1.33x1.80mm_HandSolder, F.Cu at (169.0, 133.8)
- added Coutx4_4: 22uF, Capacitor_SMD:C_1206_3216Metric_Pad1.33x1.80mm_HandSolder, F.Cu at (169.0, 131.2)
- added H1: MountingHole, MountingHole:MountingHole_3.2mm_M3_Pad_Via, F.Cu at (164.0, 23.0)
- added H1: MountingHole, MountingHole:MountingHole_3.2mm_M3_Pad_Via, F.Cu at (130.0, 23.0)
- added H3: MountingHole, MountingHole:MountingHole_3.2mm_M3_Pad_Via, F.Cu at (147.0, 150.0)
- Cout3: value 66uF -> 220uF
- L1, L3, L4: value 1uH -> 3.3uH
- L2: value 1uH -> 1.5uH
- Rsense1, Rsense4: value 1.8m -> 3m; footprint Resistor_SMD:R_1206_3216Metric_Pad1.30x1.75mm_HandSolder -> Footprints:WSLP2512-3L000
- Rsense2: value 3.6m -> 3m; footprint Resistor_SMD:R_1206_3216Metric_Pad1.30x1.75mm_HandSolder -> Footprints:WSLP2512-3L000
- Rsense3: value 5m -> 6m; footprint Resistor_SMD:R_1206_3216Metric_Pad1.30x1.75mm_HandSolder -> Footprints:WSLP2512-6L000
- moved Q3_2_3 5.21 mm to (95.9, 49.4)
- moved Q2_2 5.10 mm to (95.8, 110.6)
- moved Q4_3 4.80 mm to (99.1, 34.9), turned to 0 degrees
- moved Q3_3 4.03 mm to (95.9, 55.2)
- moved Q3_2_2 3.99 mm to (95.8, 116.1)
- moved Rfbb2 3.78 mm to (131.2, 105.0)
- moved Rfbt2 3.78 mm to (133.8, 105.0)
- moved Rfbb3 3.77 mm to (131.2, 42.0)
- moved Rfbt3 3.77 mm to (133.8, 42.0)
- moved Q4_2 3.49 mm to (99.0, 99.4), turned to 0 degrees
- moved Rfbt4 3.38 mm to (162.0, 131.2)
- moved Rfbb4 3.38 mm to (164.5, 131.2)
- moved Rfbt1 2.25 mm to (163.2, 69.2)
- moved Rfbb1 2.25 mm to (165.8, 69.2)
- moved Q3_2 2.02 mm to (95.8, 121.6)
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Connections:
- Rcsg1 pad 2: /lm5176 12v Channel 1/CSG_1 -> GND
- Rcsg2 pad 2: CSG_2 -> GND
- Rcsg3 pad 2: CSG_3 -> GND
- Rcsg4 pad 2: /lm5176 12v Channel 2/CSG_1 -> GND
- Rsense1 pad 2: /lm5176 12v Channel 1/CSG_1 -> GND
- Rsense2 pad 2: CSG_2 -> GND
- Rsense3 pad 2: CSG_3 -> GND
- Rsense4 pad 2: /lm5176 12v Channel 2/CSG_1 -> GND
Routing:
- net VOSNS_2: track 53.2 -> 75.1 mm
- net GND: track 90.5 -> 104.2 mm, vias 362 -> 398
- net Net-(U3-BIAS): track 40.0 -> 26.3 mm, vias 4 -> 2
- net VOSNS_3: track 53.4 -> 66.9 mm, vias 2 -> 1
- net Net-(U2-BIAS): track 40.0 -> 26.4 mm, vias 4 -> 2
- net /lm5176 12v Channel 2/SW2_1: track 84.2 -> 71.8 mm, vias 3 -> 5
- net SW1_2: track 54.1 -> 66.1 mm
- net VCC: track 71.8 -> 59.9 mm
- net /lm5176 12v Channel 2/BIAS_1: track 74.6 -> 86.2 mm
- net SW2_3: track 82.6 -> 71.5 mm, vias 4 -> 5
- net /lm5176 12v Channel 1/BIAS_1: track 75.0 -> 85.6 mm
- net SW2_2: track 81.6 -> 72.3 mm, vias 4 -> 5
- net Net-(U2-CS): track 10.2 -> 15.5 mm
- net /lm5176 12v Channel 1/HDRV1_1: track 25.3 -> 20.0 mm, vias 3 -> 0
- net Net-(U1-CS): track 11.3 -> 16.4 mm
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- added copper zone on F.Cu, net VOSNS_2
Other:
- board size 207.5 x 137 mm -> 208 x 137 mm
- board text added: "Power Distribution Board V3"
- board text added: "SEPT 22 2026"
- board text added: "UGRT"
- board text added: "USE XT90-S (Anti spark)"
- board text removed: "JULY 15 2026"
- board text removed: "Power Distro Board V3"

Commit message: Updated PDBV3
Parts:
- moved Cboot1_2 4.14 mm to (115.2, 130.6)
- moved Cboot2_2 4.14 mm to (112.7, 130.6)
- moved Rmode2 4.14 mm to (129.7, 128.7)
- moved Rvisns2 4.14 mm to (129.7, 131.2)
- moved Cbias1 4.14 mm to (176.0, 72.8)
- moved Cbias2 4.14 mm to (124.5, 108.2)
- moved Cbias4 4.14 mm to (175.6, 134.8)
- moved Cboot1_1 4.14 mm to (184.0, 50.2)
- moved Cboot1_4 4.14 mm to (183.8, 112.2)
- moved Cboot2_1 4.14 mm to (186.7, 50.2)
- moved Cboot2_4 4.14 mm to (186.6, 112.2)
- moved Cbulk1 4.14 mm to (189.5, 39.5)
- moved Cbulk2 4.14 mm to (110.5, 142.0)
- moved Cbulk3 4.14 mm to (110.5, 78.8)
- moved Cbulk4 4.14 mm to (188.2, 101.0)
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