File: Power Board Revisions/PDB_V3/lm5176-12v.kicad_sch (KiCad schematic)
At the start: 39 parts, among them Q1_1 NMOS, Q1_2_1 NMOS, Q2_1 NMOS, Q3_1 NMOS, Q3_2_1 NMOS, Q4_1 NMOS, U1 LM5176QPWPRQ1

Commit message: Finalized PDB V3 for first design review
Parts:
- L1: footprint Footprints:XAL1580 -> Footprints:WE-HCM_1411
Other:
- company: (none) -> University of Guelph Robotics Team
- title: (none) -> LM5176 12V Channel
Changed lines of the file:
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@@
 	(generator_version "10.0")
 	(paper "A4")
+	(title_block
+		(title "LM5176 12V Channel")
+		(date "2026-07-15")
+		(rev "1")
+		(company "University of Guelph Robotics Team")
+	)
 	(junction
 		(at 182.88 27.94)
@@
 			)
 		)
-		(property "Footprint" "Footprints:XAL1580"
+		(property "Footprint" "Footprints:WE-HCM_1411"
 			(at 157.48 45.72 0)
 			(hide yes)

Commit message: Updated PDB V3
Parts:
- Q3_1, Q3_2_1, Q4_1: footprint Footprints:CSD17575Q3 -> Footprints:IAUCN04S7L019
Changed lines of the file:
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@@
 			)
 		)
-		(property "Footprint" "Footprints:CSD17575Q3"
+		(property "Footprint" "Footprints:IAUCN04S7L019"
 			(at 185.42 31.75 0)
 			(hide yes)
@@
 			)
 		)
-		(property "Footprint" "Footprints:CSD17575Q3"
+		(property "Footprint" "Footprints:IAUCN04S7L019"
 			(at 172.72 50.8 0)
 			(hide yes)
@@
 			)
 		)
-		(property "Footprint" "Footprints:CSD17575Q3"
+		(property "Footprint" "Footprints:IAUCN04S7L019"
 			(at 172.72 35.56 0)
 			(hide yes)

Commit message: Finalized PDB V3 Rev 1
Parts:
- added Coutx1_2, Coutx1_3, Coutx1_4: 22uF, Capacitor_SMD:C_1206_3216Metric_Pad1.33x1.80mm_HandSolder, symbol Device:C
- Coutx1_1: renamed from Coutx1; value 70uF -> 22uF
- L1: value 1uH -> 3.3uH
- Rsense1: value 1.8m -> 3m; footprint Resistor_SMD:R_1206_3216Metric_Pad1.30x1.75mm_HandSolder -> Footprints:WSLP2512-3L000
Connections:
- net CSG_1 is gone; now on net GND: Rcsg1.2, Rsense1.2
- net GND: now also Coutx1_2.2, Coutx1_3.2, Coutx1_4.2
- net out_pos: now also Coutx1_2.1, Coutx1_3.1, Coutx1_4.1
Other:
- moved on the sheet: Cbias1, Coutx1_1
