File: Power Board Revisions/PDB_V3/lm5176-24v.kicad_sch (KiCad schematic)
At the start: 39 parts, among them Q1_2_3 NMOS, Q1_3 NMOS, Q2_3 NMOS, Q3_2_3 NMOS, Q3_3 NMOS, Q4_3 NMOS, U3 LM5176QPWPRQ1

Commit message: Finalized PDB V3 for first design review
Parts:
- L3: footprint Footprints:XAL1580 -> Footprints:WE-HCM_1411
Other:
- company: (none) -> University of Guelph Robotics Team
- title: (none) -> LM5176 24V Channel
Changed lines of the file:
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@@
 	(generator_version "10.0")
 	(paper "A4")
+	(title_block
+		(title "LM5176 24V Channel")
+		(date "2026-07-15")
+		(rev "1")
+		(company "University of Guelph Robotics Team")
+	)
 	(junction
 		(at 44.45 111.76)
@@
 			)
 		)
-		(property "Footprint" "Footprints:XAL1580"
+		(property "Footprint" "Footprints:WE-HCM_1411"
 			(at 147.32 41.91 0)
 			(hide yes)

Commit message: Updated PDB V3
Parts:
- Q3_2_3, Q3_3, Q4_3: footprint Footprints:CSD17575Q3 -> Footprints:IAUCN04S7L019
Changed lines of the file:
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@@
 			)
 		)
-		(property "Footprint" "Footprints:CSD17575Q3"
+		(property "Footprint" "Footprints:IAUCN04S7L019"
 			(at 167.64 31.75 0)
 			(hide yes)
@@
 			)
 		)
-		(property "Footprint" "Footprints:CSD17575Q3"
+		(property "Footprint" "Footprints:IAUCN04S7L019"
 			(at 180.34 27.94 0)
 			(hide yes)
@@
 			)
 		)
-		(property "Footprint" "Footprints:CSD17575Q3"
+		(property "Footprint" "Footprints:IAUCN04S7L019"
 			(at 167.64 46.99 0)
 			(hide yes)

Commit message: Finalized PDB V3 Rev 1
Parts:
- added Coutx3_2, Coutx3_3, Coutx3_4: 22uF, Capacitor_SMD:C_1206_3216Metric_Pad1.33x1.80mm_HandSolder, symbol Device:C
- Cout3: value 66uF -> 220uF
- Coutx3_1: renamed from Coutx3; value 70uF -> 22uF
- L3: value 1uH -> 3.3uH
- Rsense3: value 5m -> 6m; footprint Resistor_SMD:R_1206_3216Metric_Pad1.30x1.75mm_HandSolder -> Footprints:WSLP2512-6L000
Connections:
- net CSG_3 is gone; now on net GND: Rcsg3.2, Rsense3.2
- net GND: now also Coutx3_2.2, Coutx3_3.2, Coutx3_4.2
- net VOSNS_3: now also Coutx3_2.1, Coutx3_3.1, Coutx3_4.1
Other:
- moved on the sheet: Cout3, Coutx3_1, Rfbb3, Rfbt3
