File: Power Board Revisions/PDB_V3/lm5176-5v.kicad_sch (KiCad schematic)
At the start: 38 parts, among them Q1_2 NMOS, Q2_2 NMOS, Q3_2 NMOS, Q3_2_2 NMOS, Q4_2 NMOS, U2 LM5176QPWPRQ1

Commit message: Finalized PDB V3 for first design review
Parts:
- L2: footprint Footprints:XAL1580 -> Footprints:WE-HCM_1411
Other:
- company: (none) -> University of Guelph Robotics Team
- title: (none) -> LM5176 5V Channel
Changed lines of the file:
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@@
 	(generator_version "10.0")
 	(paper "A4")
+	(title_block
+		(title "LM5176 5V Channel")
+		(date "2026-07-15")
+		(rev "1")
+		(company "University of Guelph Robotics Team")
+	)
 	(junction
 		(at 76.2 102.87)
@@
 			)
 		)
-		(property "Footprint" "Footprints:XAL1580"
+		(property "Footprint" "Footprints:WE-HCM_1411"
 			(at 149.86 44.45 0)
 			(hide yes)

Commit message: Updated PDB V3
Parts:
- Q3_2, Q3_2_2, Q4_2: footprint Footprints:CSD17575Q3 -> Footprints:IAUCN04S7L019
Changed lines of the file:
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@@
 			)
 		)
-		(property "Footprint" "Footprints:CSD17575Q3"
+		(property "Footprint" "Footprints:IAUCN04S7L019"
 			(at 168.91 49.53 0)
 			(hide yes)
@@
 			)
 		)
-		(property "Footprint" "Footprints:CSD17575Q3"
+		(property "Footprint" "Footprints:IAUCN04S7L019"
 			(at 168.91 34.29 0)
 			(hide yes)
@@
 			)
 		)
-		(property "Footprint" "Footprints:CSD17575Q3"
+		(property "Footprint" "Footprints:IAUCN04S7L019"
 			(at 181.61 31.75 0)
 			(hide yes)

Commit message: Finalized PDB V3 Rev 1
Parts:
- added Coutx2_2, Coutx2_3, Coutx2_4: 22uF, Capacitor_SMD:C_1206_3216Metric_Pad1.33x1.80mm_HandSolder, symbol Device:C
- Coutx2_1: renamed from Coutx2; value 66uF -> 22uF
- L2: value 1uH -> 1.5uH
- Rsense2: value 3.6m -> 3m; footprint Resistor_SMD:R_1206_3216Metric_Pad1.30x1.75mm_HandSolder -> Footprints:WSLP2512-3L000
Connections:
- net CSG_2 is gone; now on net GND: Rcsg2.2, Rsense2.2
- net GND: now also Coutx2_2.2, Coutx2_3.2, Coutx2_4.2
- net VOSNS_2: now also Coutx2_2.1, Coutx2_3.1, Coutx2_4.1
Other:
- moved on the sheet: Cout2, Coutx2_1, Rfbb2, Rfbt2
